Commit message: changed materials to local

File: asv_zed2icamera_workspace/src/zed2i_camera/urdf/zed_macro.urdf.xacro (robot description, xacro)
@@ -16,5 +16,7 @@
 -->
 <robot xmlns:xacro="http://wiki.ros.org/xacro">
-  <xacro:include filename="$(find zed_wrapper)/urdf/include/materials.urdf.xacro" />
+  <material name="zed2i_mat">
+    <color rgba="0.25 0.25 0.25 1.0"/>
+  </material>
   <xacro:property name="M_PI"     value="3.1415926535897931" />
   <xacro:macro name="zed_camera" params="enable_gnss=false custom_baseline=0 *gnss_origin">

Commit message: fixed camera name

File: asv_zed2icamera_workspace/src/zed2i_camera/urdf/zed_macro.urdf.xacro (robot description, xacro)
@@ -22,4 +22,6 @@
   <xacro:macro name="zed_camera" params="enable_gnss=false custom_baseline=0 *gnss_origin">
     <xacro:property name="baseline" value="0.12" />
+    <xacro:property name="name" value="zed" />
+    <xacro:property name="model" value="zed2i" />
     <xacro:property name="height" value="0.03" />
     <xacro:property name="bottom_slope" value="0.0" />

Commit message: added sonar to tf

File: asv_zed2icamera_workspace/src/zed2i_camera/urdf/zed_macro.urdf.xacro (robot description, xacro)
@@ -121,4 +121,11 @@
       </joint>
     </xacro:if>
+    <!-- FAKE SONAR -->
+    <link name="base_laser_frame"/>
+    <joint name="base_laser_joint" type="fixed">
+      <origin xyz="0 0 0" rpy="-${M_PI/2} 0.0 -${M_PI/2}"/>
+      <parent link="${name}_left_camera_frame"/>
+      <child link="${name}_left_camera_optical_frame"/>
+    </joint>
   </xacro:macro>
 </robot>

Commit message: forgot a $

File: asv_zed2icamera_workspace/src/zed2i_camera/urdf/zed_macro.urdf.xacro (robot description, xacro)
@@ -126,5 +126,5 @@
       <origin xyz="0 0 0" rpy="-${M_PI/2} 0.0 -${M_PI/2}"/>
       <parent link="${name}_left_camera_frame"/>
-      <child link="$base_laser_frame"/>
+      <child link="base_laser_frame"/>
     </joint>
   </xacro:macro>
