Commit message: fixed bad child link

File: asv_zed2icamera_workspace/src/zed2i_camera/urdf/ship_descr.urdf.xacro (robot description, xacro)
@@ -17,5 +17,5 @@
 <robot name="ASV_LOYOLA_US" xmlns:xacro="http://ros.org/wiki/xacro">
   <xacro:arg name="camera_name"   default="zed" />
-  <xacro:arg name="camera_model"  default="zed" />
+  <xacro:arg name="camera_model"  default="zed2i" />
   <xacro:arg name="custom_baseline"  default="0.0" />
   <!-- If GNSS fusion is enabled the position of the antenna with respect to the camera mount point is required -->

File: asv_zed2icamera_workspace/src/zed2i_camera/urdf/zed_macro.urdf.xacro (robot description, xacro)
@@ -126,5 +126,5 @@
       <origin xyz="0 0 0" rpy="-${M_PI/2} 0.0 -${M_PI/2}"/>
       <parent link="${name}_left_camera_frame"/>
-      <child link="${name}_left_camera_optical_frame"/>
+      <child link="$base_laser_frame"/>
     </joint>
   </xacro:macro>

Commit message: added base link

File: asv_zed2icamera_workspace/src/zed2i_camera/urdf/ship_descr.urdf.xacro (robot description, xacro)
@@ -24,7 +24,13 @@
   <xacro:arg name="gnss_y" default="0.0" />
   <xacro:arg name="gnss_z" default="0.0" />
+  <link name="base_link"/>
   <xacro:include filename="$(find zed2i_camera)/urdf/zed_macro.urdf.xacro" />
   <xacro:zed_camera custom_baseline="$(arg custom_baseline)" enable_gnss="$(arg enable_gnss)">
 	    <origin xyz="$(arg gnss_x) $(arg gnss_y) $(arg gnss_z)" rpy="0 0 0"/>
   </xacro:zed_camera>
+  <joint name="base_camera_joint" type="fixed">
+      <origin xyz="0 2.0 0" rpy="0.0 0.0 0.0"/>
+      <parent link="base_link"/>
+      <child link="${name}_camera_link"/>
+    </joint>
 </robot>

Commit message: changed config to reach syncronization

File: asv_zed2icamera_workspace/src/zed2i_camera/urdf/ship_descr.urdf.xacro (robot description, xacro)
@@ -32,5 +32,5 @@
       <origin xyz="0 2.0 0" rpy="0.0 0.0 0.0"/>
       <parent link="base_link"/>
-      <child link="${name}_camera_link"/>
+      <child link="${camera_name}_camera_link"/>
     </joint>
 </robot>

Commit message: updated parameters to avoid 2 odoms

File: asv_zed2icamera_workspace/src/zed2i_camera/urdf/ship_descr.urdf.xacro (robot description, xacro)
@@ -32,5 +32,5 @@
       <origin xyz="0 2.0 0" rpy="0.0 0.0 0.0"/>
       <parent link="base_link"/>
-      <child link="${camera_name}_camera_link"/>
+      <child link="$(arg camera_name)_camera_link"/>
     </joint>
 </robot>

Commit message: new link tf

File: asv_zed2icamera_workspace/src/zed2i_camera/urdf/ship_descr.urdf.xacro (robot description, xacro)
@@ -33,4 +33,9 @@
       <parent link="base_link"/>
       <child link="$(arg camera_name)_camera_link"/>
-    </joint>
+  </joint>
+  <joint name="robot_joint" type="fixed">
+      <origin xyz="0 2.0 0" rpy="0.0 0.0 0.0"/>
+      <parent link="odom"/>
+      <child link="base_link"/>
+  </joint>
 </robot>

Commit message: changed link ref for base link

File: asv_zed2icamera_workspace/src/zed2i_camera/urdf/ship_descr.urdf.xacro (robot description, xacro)
@@ -31,10 +31,5 @@
   <joint name="base_camera_joint" type="fixed">
       <origin xyz="0 2.0 0" rpy="0.0 0.0 0.0"/>
-      <parent link="base_link"/>
-      <child link="$(arg camera_name)_camera_link"/>
-  </joint>
-  <joint name="robot_joint" type="fixed">
-      <origin xyz="0 2.0 0" rpy="0.0 0.0 0.0"/>
-      <parent link="odom"/>
+      <parent link="$(arg camera_name)_camera_link"/>
       <child link="base_link"/>
   </joint>
